Commit message: remove the lift, partially

File: urdf/vector.xacro (robot description, xacro)
@@ -69,8 +69,8 @@
     <visual>
       <geometry>
-        <mesh filename="package://anki_description/meshes/vector_lift.dae"/>
+        <mesh filename="package://anki_description/meshes/vector_lift.dae" />
       </geometry>
     </visual>
-    <collision>
+    <!-- <collision>
       <origin rpy="0 0 0" xyz="0.062 0.0 -0.015"/>
       <geometry>
@@ -85,5 +85,5 @@
       <mass value="0.05"/>
       <xacro:box_inertia m="0.05" x="0.0075" y="0.05" z="0.025"/>
-    </inertial>
+    </inertial> -->
   </link>
   <gazebo reference="full_lift">
